File: XIAO Family/XIAO.kicad_sch (KiCad schematic)
At the start: 22 parts, among them U1 XIAO-SAMD21-SMD, U10 XIAO-ESP32-C6-DIP, U11 XIAO-ESP32-S3-DIP, U12 XIAO-ESP32-C3-DIP, U13 XIAO-RP2350-SMD, U14 XIAO-R4-SMD, U15 XIAO-Add-On, U16 XIAO-RP2350-DIP, U17 XIAO-R4-DIP, U18 XIAO-ESP32-C5-SMD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

Commit message: Update XIAO Series family images and files
Parts:
- removed U15: XIAO-Add-On, Seeed_Studio_XIAO_Series:XIAO-Add-On, symbol MCU_SEEED_XIAO_Series:XIAO-Add-on
- U10: footprint MCU_SEEED_XIAO_Series:XIAO-ESP32-C6-DIP -> Seeed_Studio_XIAO_Series:XIAO-ESP32-C6-DIP; symbol MCU_SEEED_XIAO_Series:XIAO-ESP32-C6-DIP -> Seeed_Studio_XIAO_Series:XIAO-ESP32-C6-DIP
- U11: footprint MCU_SEEED_XIAO_Series:XIAO-ESP32-S3-DIP -> Seeed_Studio_XIAO_Series:XIAO-ESP32-S3-DIP; symbol MCU_SEEED_XIAO_Series:XIAO-ESP32-S3-DIP -> Seeed_Studio_XIAO_Series:XIAO-ESP32-S3-DIP
- U12: footprint MCU_SEEED_XIAO_Series:XIAO-ESP32-C3-DIP -> Seeed_Studio_XIAO_Series:XIAO-ESP32-C3-DIP; symbol MCU_SEEED_XIAO_Series:XIAO-ESP32-C3-DIP -> Seeed_Studio_XIAO_Series:XIAO-ESP32-C3-DIP
- U13: footprint MCU_SEEED_XIAO_Series:XIAO-RP2350-SMD -> Seeed_Studio_XIAO_Series:XIAO-RP2350-SMD; symbol MCU_SEEED_XIAO_Series:XIAO-RP2350-SMD -> Seeed_Studio_XIAO_Series:XIAO-RP2350-SMD
- U16: footprint MCU_SEEED_XIAO_Series:XIAO-RP2350-DIP -> Seeed_Studio_XIAO_Series:XIAO-RP2350-DIP; symbol MCU_SEEED_XIAO_Series:XIAO-RP2350-DIP -> Seeed_Studio_XIAO_Series:XIAO-RP2350-DIP
- U2: footprint MCU_SEEED_XIAO_Series:XIAO-RP2040-SMD -> Seeed_Studio_XIAO_Series:XIAO-RP2040-SMD; symbol MCU_SEEED_XIAO_Series:XIAO-RP2040-SMD -> Seeed_Studio_XIAO_Series:XIAO-RP2040-SMD
- U3: footprint MCU_SEEED_XIAO_Series:XIAO-nRF52840-SMD -> Seeed_Studio_XIAO_Series:XIAO-nRF52840-SMD; symbol MCU_SEEED_XIAO_Series:XIAO-nRF52840-SMD -> Seeed_Studio_XIAO_Series:XIAO-nRF52840-SMD
- U5: footprint MCU_SEEED_XIAO_Series:XIAO-RP2040-DIP -> Seeed_Studio_XIAO_Series:XIAO-RP2040-DIP; symbol MCU_SEEED_XIAO_Series:XIAO-RP2040-DIP -> Seeed_Studio_XIAO_Series:XIAO-RP2040-DIP
- U6: footprint MCU_SEEED_XIAO_Series:XIAO-nRF52840-DIP -> Seeed_Studio_XIAO_Series:XIAO-nRF52840-DIP; symbol MCU_SEEED_XIAO_Series:XIAO-nRF52840-DIP -> Seeed_Studio_XIAO_Series:XIAO-nRF52840-DIP
- U7: footprint MCU_SEEED_XIAO_Series:XIAO-ESP32-C6-SMD -> Seeed_Studio_XIAO_Series:XIAO-ESP32-C6-SMD; symbol MCU_SEEED_XIAO_Series:XIAO-ESP32-C6-SMD -> Seeed_Studio_XIAO_Series:XIAO-ESP32-C6-SMD
- U8: footprint MCU_SEEED_XIAO_Series:XIAO-ESP32-C3-SMD -> Seeed_Studio_XIAO_Series:XIAO-ESP32-C3-SMD; symbol MCU_SEEED_XIAO_Series:XIAO-ESP32-C3-SMD -> Seeed_Studio_XIAO_Series:XIAO-ESP32-C3-SMD
- U9: footprint MCU_SEEED_XIAO_Series:XIAO-ESP32-S3-SMD -> Seeed_Studio_XIAO_Series:XIAO-ESP32-S3-SMD; symbol MCU_SEEED_XIAO_Series:XIAO-ESP32-S3-SMD -> Seeed_Studio_XIAO_Series:XIAO-ESP32-S3-SMD
Other:
- moved on the sheet: U14, U17, U19, U20, U21, U22
